File: 1_ega/3_esquematico_pcb/electronic_load/electronic_load.kicad_sch (KiCad schematic)
At the start: 54 parts, among them J1 Encoder, J10 5V, J11 LOAD, J12 Memoria SD, J13 LCD, J14 INA219, J15 VCC, J17 EGB_I2C, J18 EGB_UART, J2 RTC_I2C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

Commit message: pcb small changes
Parts:
- L1: value 170uH -> 220uH
Changed lines of the file:
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@@
 			)
 		)
-		(property "Value" "170uH"
+		(property "Value" "220uH"
 			(at 252.73 124.4599 0)
 			(effects
