File: 1_ega/3_esquematico_pcb/electronic_load/electronic_load.kicad_pcb (KiCad board)
At the start: 2 copper layers, 100 x 100 mm, 59 parts, among them J1 Encoder, J10 5V, J11 LOAD, J12 Memoria SD, J13 LCD, J14 INA219, J15 VCC, J17 EGB_I2C, J18 EGB_UART, J2 RTC_I2C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

Commit message: Update last version of pcb
Parts:
- added RV1: 1k, Connector_PinHeader_2.54mm:PinHeader_1x03_P2.54mm_Vertical, F.Cu at (41.9, 45.7)
- added RV2: 1k, Connector_PinHeader_2.54mm:PinHeader_1x03_P2.54mm_Vertical, F.Cu at (68.4, 99.4)
- moved R18 10.5 mm to (82.3, 93.7), turned to 180 degrees
- moved J4 6.28 mm to (84.8, 88.2), turned to -90 degrees
- moved R11 2.46 mm to (64.1, 91.2)
- moved C1 2.42 mm to (42.0, 40.2), turned to 90 degrees
- moved R12 2.21 mm to (75.3, 87.4)
- moved R25 2.16 mm to (32.9, 45.7)
- moved J9 0.97 mm to (44.3, 68.1)
- moved R22 0.91 mm to (43.3, 49.7)
- moved R23 0.89 mm to (43.2, 63.5)
- moved R6 0.87 mm to (60.9, 73.8)
- moved C2 0.80 mm to (60.9, 87.7)
- moved R24 0.47 mm to (38.3, 49.4)
- moved R15 0.46 mm to (45.0, 89.9)
- moved D2 0.18 mm to (93.0, 99.2)
Connections:
- R12 pad 2: Net-(U1A--) -> Net-(R12-Pad2)
- R25 pad 1: Net-(U2-Vfb) -> Net-(R25-Pad1)
Routing:
- net Net-(U1A--): track 18.9 -> 30.3 mm
- net Net-(R12-Pad2): track 0.00 -> 8.29 mm
- net Net-(R11-Pad2): track 16.2 -> 23.3 mm
- net Net-(R25-Pad1): track 0.00 -> 6.44 mm
- net +5V: track 189.2 -> 194.1 mm
- net MOS_GATE: track 22.2 -> 19.6 mm
- net Net-(D2-A): track 61.1 -> 59.5 mm
- net Net-(U2-DC): track 8.04 -> 8.93 mm
- net TEMP_DIODE: track 104.4 -> 105.2 mm
- net MOS_DRAIN: track 49.7 -> 48.9 mm
- net Net-(U1A-+): track 14.0 -> 13.4 mm

Commit message: update pcb to last version
Parts:
- moved J2 4.15 mm to (69.8, 66.3)
- moved R21 1.05 mm to (56.1, 77.6)
- moved R11 0.69 mm to (63.5, 91.1)
- moved Q3 0.25 mm to (48.3, 85.8)
- moved Q4 0.25 mm to (41.0, 85.8)
Routing:
- net +3V3: track 134.7 -> 140.2 mm
- net RTC_32K: track 12.5 -> 9.66 mm
- net RTC_SQW: track 16.3 -> 14.2 mm
- net I2C_SCL: track 64.8 -> 66.8 mm
- net TEMP_DIODE: track 105.2 -> 103.3 mm
- net I2C_SDA: track 68.6 -> 70.3 mm
- net GND: track 211.2 -> 210.3 mm

Commit message: chore: update PCB pdf to final version
Parts:
- C6: value 470uF -> 330uF
- J1: footprint Connector_PinHeader_2.54mm:PinHeader_1x05_P2.54mm_Vertical -> Connector_Molex:Molex_KK-254_AE-6410-05A_1x05_P2.54mm_Vertical
- R11: value 20k -> 5.1k
- R12: value 5.1k -> 12k
- R26: value 1k5 -> 2.2k
- R28: value 200R -> 150R
- RV2: value 1k -> 5k
- moved J1 0.16 mm to (46.7, 28.0), turned to 0 degrees
