File: 1_ega/3_esquematico_pcb/electronic_load_v2/electronic_load_v2.kicad_pcb (KiCad board)
At the start: 2 copper layers, 100 x 62.5 mm, 57 parts, among them J1 Encoder, J10 5V, J11 LOAD, J12 Memoria SD, J13 LCD, J15 VCC, J17 EGB_I2C, J2 RTC_I2C, J6 RPico PWR, Q1 IRF540N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

Commit message: chore: pcb v1 10x5 con R y C smd. INA modulo
Parts:
- removed D5: LED_R, LED_THT:LED_D5.0mm
- removed J10: 5V, TerminalBlock_Phoenix:TerminalBlock_Phoenix_MKDS-1,5-2-5.08_1x02_P5.08mm_Horizontal
- removed J2: RTC_I2C, Connector_PinSocket_2.54mm:PinSocket_1x06_P2.54mm_Vertical
- removed R28: 150R, Resistor_SMD:R_0805_2012Metric_Pad1.20x1.40mm_HandSolder
- removed U4: TL072, Package_DIP:DIP-8_W7.62mm_LongPads
- added C7: 330nF, Capacitor_SMD:C_0805_2012Metric_Pad1.18x1.45mm_HandSolder, B.Cu at (79.1, 102.1)
- added J16: RTC, Connector_PinHeader_2.54mm:PinHeader_1x04_P2.54mm_Vertical, F.Cu at (101.5, 95.9)
- added J3: GND, Connector_PinHeader_2.54mm:PinHeader_1x02_P2.54mm_Vertical, F.Cu at (112.0, 60.1)
- added J7: GND, Connector_PinHeader_2.54mm:PinHeader_1x02_P2.54mm_Vertical, F.Cu at (29.0, 103.8)
- added J8: 5V, Connector_PinHeader_2.54mm:PinHeader_1x02_P2.54mm_Vertical, F.Cu at (98.0, 103.6)
- added R30: 3.3k, Resistor_SMD:R_1206_3216Metric_Pad1.30x1.75mm_HandSolder, B.Cu at (44.8, 104.3)
- added TP1: MOS_GATE, Connector_Pin:Pin_D0.7mm_L6.5mm_W1.8mm_FlatFork, F.Cu at (32.6, 98.9)
- added TP2: MOS_SK, Connector_Pin:Pin_D0.7mm_L6.5mm_W1.8mm_FlatFork, F.Cu at (49.0, 101.3)
- added TP3: MOS_OFFSET, Connector_Pin:Pin_D0.7mm_L6.5mm_W1.8mm_FlatFork, F.Cu at (49.0, 104.3)
- added TP4: T_DIODE, Connector_Pin:Pin_D0.7mm_L6.5mm_W1.8mm_FlatFork, F.Cu at (57.1, 82.7)
- added TP5: Isense, Connector_Pin:Pin_D0.7mm_L6.5mm_W1.8mm_FlatFork, F.Cu at (32.9, 83.7)
- C1: value 10uF -> 100uF; footprint Capacitor_THT:CP_Radial_D6.3mm_P2.50mm -> Capacitor_THT:CP_Radial_D5.0mm_P2.50mm
- C6: value 10uF -> 100nF; footprint Capacitor_THT:CP_Radial_D6.3mm_P2.50mm -> Capacitor_SMD:C_0805_2012Metric_Pad1.18x1.45mm_HandSolder; moved to B.Cu
- Q1: footprint Package_TO_SOT_THT:TO-220F-3_Horizontal_TabUp -> Package_TO_SOT_THT:TO-220-3_Vertical
- R11, R12, R14, R15, R16, R17, R18, R19, R22, R23, R24, R25, R26, R27, R29, R6, R7: footprint Resistor_SMD:R_0805_2012Metric_Pad1.20x1.40mm_HandSolder -> Resistor_SMD:R_1206_3216Metric_Pad1.30x1.75mm_HandSolder
- R20, R21: footprint Resistor_SMD:R_0805_2012Metric_Pad1.20x1.40mm_HandSolder -> Resistor_THT:R_Axial_DIN0207_L6.3mm_D2.5mm_P10.16mm_Horizontal; moved to F.Cu
- RV1, RV2: footprint Connector_PinHeader_2.54mm:PinHeader_1x03_P2.54mm_Vertical -> Potentiometer_THT:Potentiometer_Bourns_3296W_Vertical
- U1: value TL072 -> LM324; footprint Package_DIP:DIP-8_W7.62mm_LongPads -> Package_DIP:DIP-14_W7.62mm_Socket
- moved HS1 130.2 mm to (29.2, 92.2), turned to -90 degrees
- moved J17 88.9 mm to (112.3, 66.4), turned to 90 degrees
- moved SW1 84.0 mm to (105.7, 62.6), turned to 0 degrees
- moved C3 81.5 mm to (107.2, 67.7), turned to 0 degrees
- moved SW2 79.9 mm to (99.2, 62.5), turned to 0 degrees
- moved C4 78.7 mm to (102.9, 67.7), turned to 180 degrees
- moved D2 76.5 mm to (25.1, 96.3), turned to 90 degrees
- moved U2 73.9 mm to (27.4, 61.1), turned to -90 degrees
- moved J6 73.5 mm to (116.7, 97.3), turned to 180 degrees
- moved R26 70.3 mm to (36.0, 83.7), turned to -90 degrees
- moved R29 63.7 mm to (39.2, 83.7), turned to 90 degrees
- moved J1 63.5 mm to (67.4, 62.5), turned to 0 degrees
- moved D4 61.6 mm to (110.0, 105.5)
- moved R27 60.1 mm to (106.4, 102.5)
- moved R14 59.6 mm to (45.6, 85.2), turned to 180 degrees
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Connections:
- A1 pad 10: BTN_STOP -> SPI0_TX
- A1 pad 11: TX_EGB -> SPI0_CS
- A1 pad 12: RX_EGB -> unconnected-(A1-GPIO9-Pad12)
- A1 pad 16: ENC_CLK -> unconnected-(A1-GPIO12-Pad16)
- A1 pad 17: ENC_DT -> ENC_SW
- A1 pad 19: ENC_SW -> ENC_DT
- A1 pad 20: unconnected-(A1-GPIO15-Pad20) -> ENC_CLK
- A1 pad 21: SPI0_RX -> MOS_EN
- A1 pad 22: SPI0_CS -> MOS_PWM
- A1 pad 24: SPI0_CLK -> I2C_SDA
- A1 pad 25: SPI0_TX -> I2C_SCL
- A1 pad 26: MOS_EN -> unconnected-(A1-GPIO20-Pad26)
- A1 pad 27: MOS_PWM -> unconnected-(A1-GPIO21-Pad27)
- A1 pad 31: I2C_SDA -> TEMP_DIODE
- A1 pad 32: I2C_SCL -> unconnected-(A1-GPIO27_ADC1-Pad32)
- A1 pad 33: unconnected-(A1-AGND-Pad33) -> GND
- A1 pad 34: TEMP_DIODE -> unconnected-(A1-GPIO28_ADC2-Pad34)
- A1 pad 4: unconnected-(A1-GPIO2-Pad4) -> BTN_MENU
- A1 pad 6: unconnected-(A1-GPIO4-Pad6) -> BTN_STOP
- A1 pad 7: LED_ACTIVE -> SPI0_RX
- A1 pad 9: BTN_MENU -> SPI0_CLK
- C6 pad 1: +5V -> GND
- C6 pad 2: GND -> +5V
- J1 pad 1: GND -> ENC_CLK
- J1 pad 2: +3V3 -> ENC_DT
- J1 pad 4: ENC_DT -> +3V3
- J1 pad 5: ENC_CLK -> GND
- J12 pad 3: SPI0_RX -> SPI0_CS
- J12 pad 6: SPI0_CS -> SPI0_RX
- J17 pad 1: EGB_TX_SDA -> EGB_RX_SCL
- J17 pad 2: EGB_RX_SCL -> EGB_TX_SDA
- R14 pad 1: Net-(U4A--) -> Net-(U1B--)
- R15 pad 1: Net-(U4A--) -> Net-(U1B--)
- R16 pad 1: GND -> MOS_OFFSET
- R16 pad 2: MOS_OFFSET -> MOS_EN
- R17 pad 2: Net-(U1B-+) -> Net-(U1D-+)
- R22 pad 2: Net-(U1B-+) -> Net-(U1D-+)
- R23 pad 1: Net-(U1B--) -> Net-(U1D--)
- R24 pad 2: Net-(U1B--) -> Net-(U1D--)
- R25 pad 2: Net-(U4B-+) -> Net-(U1C-+)
- R26 pad 2: Net-(U4B--) -> Net-(U1C--)
- R29 pad 1: Net-(U4B--) -> Net-(U1C--)
- RV2 pad 1: MOS_EN -> Net-(R30-Pad1)
- RV2 pad 2: MOS_OFFSET -> Net-(R30-Pad1)
- RV2 pad 3: MOS_OFFSET -> GND
- U1 pad 4: GND -> VCC
- U1 pad 5: Net-(U1B-+) -> Net-(D2-A)
- U1 pad 7: MOS_GATE -> TEMP_DIODE
- U1 pad 8: VCC -> Io_sens
Routing:
- net GND: track 0.00 -> 125.2 mm
- net +3V3: track 203.7 -> 133.0 mm
- net TEMP_DIODE: track 2.51 -> 47.2 mm, vias 0 -> 2
- net LOAD+: track 62.7 -> 29.4 mm
- net VCC: track 14.9 -> 47.0 mm
- net Net-(D2-A): track 35.6 -> 66.4 mm
- net I2C_SDA: track 73.7 -> 96.9 mm
- net I2C_SCL: track 110.7 -> 89.3 mm
- net I_sens: track 9.43 -> 30.5 mm
- net MOS_OFFSET: track 9.25 -> 29.6 mm
- net +5V: track 28.4 -> 44.1 mm
- net Net-(U4B-+): track 15.3 -> 0.00 mm
- net MOS_EN: track 23.3 -> 12.0 mm
- net MOS_PWM: track 10.1 -> 19.9 mm
- net MOS_DRAIN: track 33.4 -> 42.5 mm
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Other:
- board size 100 x 62.5 mm -> 100 x 50 mm

Commit message: chore: minimal revision
Parts:
- moved TP3 5.83 mm to (54.9, 104.2)
- moved R21 2.85 mm to (70.3, 75.7)
- moved R20 2.85 mm to (70.4, 79.0)
- moved Q3 2.78 mm to (52.3, 78.6)
- moved Q4 2.74 mm to (52.3, 73.5)
- moved C1 1.92 mm to (73.5, 96.4), turned to 0 degrees
- moved R30 1.76 mm to (45.0, 102.5), turned to 90 degrees
- moved RV2 1.37 mm to (41.0, 103.2)
- moved J7 1.18 mm to (29.6, 104.9)
- moved SW3 0.52 mm to (73.4, 103.1)
- moved J15 0.50 mm to (62.5, 102.3)
- moved U2 0.39 mm to (27.4, 61.5)
- moved R1 0.35 mm to (43.3, 77.9)
Routing:
- net GND: track 125.2 -> 118.5 mm
- net Net-(D2-A): track 66.4 -> 60.5 mm
- net I2C_SDA: track 96.9 -> 100.5 mm
- net I2C_SCL: track 89.3 -> 92.3 mm
- net Net-(Q3-B): track 14.0 -> 11.7 mm
- net +3V3: track 133.0 -> 131.1 mm
- net MOS_OFFSET: track 29.6 -> 28.4 mm
- net Net-(Q4-E): track 5.39 -> 4.56 mm
- net Net-(Q3-E): track 3.64 -> 2.97 mm
- net VCC: track 47.0 -> 46.4 mm
- net Net-(R30-Pad1): track 6.63 -> 7.14 mm

Commit message: perf: ajustes en pistas y clearance para cnc
Parts:
- added C8: 0.1uF, Capacitor_SMD:C_0805_2012Metric_Pad1.18x1.45mm_HandSolder, B.Cu at (33.3, 69.0)
- added R28: 1k, Resistor_SMD:R_1206_3216Metric_Pad1.30x1.75mm_HandSolder, B.Cu at (37.7, 64.7)
- R11: value 22k -> 10k
- R12: value 10k -> 4.7k
- R14: value 5.1k -> 12k
- R15: value 20k -> 47k
- R16: value 4.7k -> 1k
- R19: value 5.1k -> 4.7k
- R27: footprint Resistor_SMD:R_1206_3216Metric_Pad1.30x1.75mm_HandSolder -> Resistor_SMD:R_0805_2012Metric_Pad1.20x1.40mm_HandSolder
- R30: value 3.3k -> 1k
- U2: value module_ina219 -> INA219AxD; footprint usini_sensors:module_ina219 -> Package_SO:SOIC-8_3.9x4.9mm_P1.27mm; moved to B.Cu
- moved U2 14.7 mm to (37.4, 72.2), turned to 90 degrees
- moved R27 0.41 mm to (106.4, 102.1)
- moved R22 0.36 mm to (44.7, 96.8)
Connections:
- U2 pad 1: +3V3 -> GND
- U2 pad 3: I2C_SCL -> I2C_SDA
- U2 pad 4: I2C_SDA -> I2C_SCL
- U2 pad 5: MOS_DRAIN -> +3V3
- U2 pad 6: LOAD+ -> GND
Routing:
- net I2C_SDA: track 100.5 -> 88.6 mm
- net LOAD+: track 29.8 -> 19.3 mm
- net GND: track 118.5 -> 128.4 mm
- net MOS_DRAIN: track 42.2 -> 50.1 mm
- net +3V3: track 131.1 -> 138.0 mm
- net I2C_SCL: track 92.3 -> 85.5 mm
- net Net-(D2-A): track 60.5 -> 63.1 mm
- net I_sens: track 30.8 -> 30.2 mm

Commit message: fix: footprint de R shunt. chore: separar los componentes en la zona del operacional
Parts:
- added R31: 1k, Resistor_SMD:R_0805_2012Metric_Pad1.20x1.40mm_HandSolder, B.Cu at (59.4, 65.0)
- added R32: 1k, Resistor_SMD:R_0805_2012Metric_Pad1.20x1.40mm_HandSolder, B.Cu at (59.4, 62.9)
- J17: value EGB_I2C -> EGB
- R1: value E100 -> R100; footprint Resistor_THT:R_Axial_DIN0309_L9.0mm_D3.2mm_P12.70mm_Horizontal -> Resistor_THT:R_Axial_DIN0922_L20.0mm_D9.0mm_P25.40mm_Horizontal
- R20, R21: footprint Resistor_THT:R_Axial_DIN0207_L6.3mm_D2.5mm_P10.16mm_Horizontal -> Resistor_THT:R_Axial_DIN0207_L6.3mm_D2.5mm_P7.62mm_Horizontal
- R28: value 1k -> R100; footprint Resistor_SMD:R_1206_3216Metric_Pad1.30x1.75mm_HandSolder -> electronic_load:R_shunt_ina219
- moved C8 31.0 mm to (63.3, 61.5)
- moved U2 17.5 mm to (53.2, 64.5), turned to 180 degrees
- moved R1 15.1 mm to (29.9, 84.9)
- moved TP3 14.1 mm to (63.0, 92.7)
- moved TP2 13.9 mm to (59.9, 92.7)
- moved J11 13.9 mm to (43.0, 62.6)
- moved RV1 12.3 mm to (51.8, 103.9), turned to 0 degrees
- moved TP5 10.0 mm to (40.5, 77.1)
- moved TP1 8.99 mm to (41.6, 99.0)
- moved R16 6.83 mm to (63.1, 87.9)
- moved R11 6.63 mm to (57.2, 96.6), turned to 90 degrees
- moved R7 4.74 mm to (57.3, 88.0)
- moved R15 4.59 mm to (57.4, 82.4)
- moved TP4 3.90 mm to (54.2, 80.2)
- moved R24 3.85 mm to (40.1, 89.5), turned to -90 degrees
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Connections:
- J11 pad 1: GND -> LOAD+
- J11 pad 2: LOAD+ -> GND
- U2 pad 1: GND -> Net-(U2-A1)
- U2 pad 2: GND -> Net-(U2-A0)
Routing:
- net GND: track 128.4 -> 70.1 mm
- net I2C_SCL: track 85.5 -> 66.7 mm
- net I_sens: track 30.2 -> 12.8 mm
- net +3V3: track 138.0 -> 122.5 mm
- net Net-(D2-A): track 63.1 -> 48.5 mm
- net MOS_SK: track 11.7 -> 24.9 mm
- net I2C_SDA: track 88.6 -> 76.9 mm
- net MOS_DRAIN: track 50.1 -> 61.0 mm
- net LOAD+: track 19.3 -> 13.0 mm
- net Io_sens: track 11.4 -> 5.97 mm
- net MOS_OFFSET: track 28.4 -> 33.3 mm
- net MOS_EN: track 12.0 -> 7.45 mm
- net Net-(U1D-+): track 6.56 -> 10.8 mm
- net Net-(R12-Pad1): track 12.1 -> 8.18 mm
- net Net-(U1B--): track 6.38 -> 9.86 mm
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
Commit message: add: change Rsense to ina smd size
Parts:
- R1: footprint Resistor_THT:R_Axial_DIN0922_L20.0mm_D9.0mm_P25.40mm_Horizontal -> electronic_load:R_shunt_ina219; moved to B.Cu
- R17, R22, R23, R24: value 100k -> 47k
- R20, R21: footprint Resistor_THT:R_Axial_DIN0207_L6.3mm_D2.5mm_P7.62mm_Horizontal -> Resistor_THT:R_Axial_DIN0207_L6.3mm_D2.5mm_P10.16mm_Horizontal
- R31, R32: footprint Resistor_SMD:R_0805_2012Metric_Pad1.20x1.40mm_HandSolder -> Resistor_SMD:R_1206_3216Metric_Pad1.30x1.75mm_HandSolder
- moved J7 49.3 mm to (61.8, 66.1), turned to 180 degrees
- moved R1 11.1 mm to (34.0, 74.5)
- moved D2 7.49 mm to (26.6, 89.3)
- moved HS1 7.06 mm to (30.5, 85.7)
- moved Q1 7.06 mm to (34.1, 88.3)
- moved TP1 6.80 mm to (34.9, 98.7)
- moved U2 6.68 mm to (46.5, 64.8)
- moved C5 6.17 mm to (57.3, 93.0)
- moved R28 6.07 mm to (33.6, 67.9)
- moved J11 6.06 mm to (36.9, 62.6)
- moved R32 5.84 mm to (53.5, 62.9)
- moved R31 5.83 mm to (53.5, 65.1)
- moved C8 5.33 mm to (58.0, 61.4)
- moved R19 4.77 mm to (43.5, 70.6), turned to 180 degrees
- moved R25 3.89 mm to (39.2, 85.4)
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Connections:
- A1 pad 24: I2C_SDA -> unconnected-(A1-GPIO18-Pad24)
- A1 pad 31: TEMP_DIODE -> I2C_SDA
- A1 pad 32: unconnected-(A1-GPIO27_ADC1-Pad32) -> TEMP_DIODE
- Q1 pad 1: Net-(Q1-G) -> MOS_GATE
- R18 pad 1: Net-(Q1-G) -> MOS_GATE
- R18 pad 2: MOS_GATE -> Net-(R18-Pad2)
- R23 pad 2: MOS_GATE -> Net-(R18-Pad2)
- U1 pad 14: MOS_GATE -> Net-(R18-Pad2)
Routing:
- net GND: track 70.1 -> 80.4 mm
- net Net-(D2-A): track 48.5 -> 38.6 mm
- net MOS_DRAIN: track 61.0 -> 53.4 mm
- net MOS_SK: track 24.9 -> 18.9 mm
- net Net-(R18-Pad2): track 0.00 -> 5.92 mm
- net I2C_SCL: track 66.7 -> 71.8 mm
- net I2C_SDA: track 76.9 -> 81.7 mm
- net Net-(Q1-G): track 4.60 -> 0.00 mm
- net Net-(U1B--): track 9.86 -> 5.81 mm
- net Net-(U1C-+): track 5.96 -> 2.85 mm
- net Net-(Q3-E): track 5.14 -> 2.19 mm
- net MOS_PWM: track 16.8 -> 14.0 mm
- net I_sens: track 12.8 -> 10.1 mm
- net Net-(D4-A): track 3.67 -> 6.41 mm
- net Net-(Q4-E): track 6.38 -> 3.65 mm
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
Commit message: chore: add name and logo
Parts:
- added G***: LOGO, LOGO, B.Cu at (27.3, 97.6)
- moved J13 1.25 mm to (93.4, 95.9)
- moved J8 1.25 mm to (99.3, 103.6)
- moved U3 1.14 mm to (86.5, 103.1)
- moved J16 0.76 mm to (102.2, 96.0)
- moved SW3 0.58 mm to (72.8, 103.0)
- moved J15 0.32 mm to (62.2, 102.3)
- moved R1 0.15 mm to (34.1, 74.7)
Connections:
- A1 pad 24: unconnected-(A1-GPIO18-Pad24) -> I2C_SDA
- A1 pad 31: I2C_SDA -> TEMP_DIODE
- A1 pad 32: TEMP_DIODE -> unconnected-(A1-GPIO27_ADC1-Pad32)
Routing:
- net GND: track 80.4 -> 180.5 mm
- net +3V3: track 121.9 -> 127.4 mm
- net +5V: track 44.6 -> 45.9 mm
- net I2C_SDA: track 81.7 -> 82.5 mm
- net Net-(D2-A): track 38.6 -> 39.4 mm
- net I2C_SCL: track 71.8 -> 72.4 mm
- net TEMP_DIODE: track 47.2 -> 47.8 mm
Other:
- board text added: "Pablo G. TD3 EGA 2025"
