File: 1_ega/3_esquematico_pcb/electronic_load_v2/electronic_load_v2.kicad_sch (KiCad schematic)
At the start: 67 parts, among them J1 Encoder, J11 LOAD, J12 Memoria SD, J13 LCD, J15 VCC, J16 RTC, J17 EGB, J3 GND, J6 RPico PWR, J7 GND, J8 5V, Q1 IRF540N, Q3 BC327, Q4 BC327, SW1 BTN_MENU, SW2 BTN_STOP, SW3 SW_PWR, U1 LM324, U2 INA219AxD, U3 LM7805_TO220

Commit message: feat: avances ajuste de filtro Sallen Key
Parts:
- C2: value 47nF -> 4.7nF
- C5: value 100nF -> 10nF
- R6, R7: value 4.7k -> 47k
Changed lines of the file:
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@@
 			)
 		)
-		(property "Value" "4.7k"
+		(property "Value" "47k"
 			(at 224.79 29.21 90)
 			(effects
@@
 			)
 		)
-		(property "Value" "4.7k"
+		(property "Value" "47k"
 			(at 214.63 29.21 90)
 			(effects
@@
 			)
 		)
-		(property "Value" "100nF"
+		(property "Value" "10nF"
 			(at 237.7441 17.78 90)
 			(effects
@@
 			)
 		)
-		(property "Value" "47nF"
+		(property "Value" "4.7nF"
 			(at 226.06 38.0999 0)
 			(effects
